File: hdw/PIC32MZ_ETH_Demo/GPIO.sch (KiCad schematic (older format))
At the start: 0 parts

Commit message: More schematic tweaks, followed PHY design guide
Parts:
- added C1001, C1002, C1003: 0.1uF, Capacitors_SMD:C_0402, symbol Custom_Library:C_Custom
- added D1001, D1002: Green, LEDs:LED_0603, symbol Device:LED
- added R1001, R1003, R1005: 10k, Resistors_SMD:R_0402, symbol Custom_Library:R_Custom
- added R1002, R1004: 1k, Resistors_SMD:R_0402, symbol Custom_Library:R_Custom
- added SW1001: GPIO_SW, Buttons_Switches_THT:SW_PUSH_6mm, symbol Switch:SW_Push
- added U1001, U1003: 74LVC1G97, Package_TO_SOT_SMD:SOT-363_SC-70-6, symbol Custom_Library:74LVC1G97_Power_NOT
- added U1002: MAX6816, Package_TO_SOT_SMD:SOT-143, symbol Interface:MAX6816
Connections:
- new net: D1001.1 (K), U1001.4
- new net: D1001.2 (A), R1002.2
- new net: D1002.1 (K), U1003.4
- new net: D1002.2 (A), R1004.2
- new net: SW1001.2, U1002.2 (IN)
- new net +3V3: C1001.1, C1002.1, C1003.1, R1002.1, R1004.1, R1005.1, U1001.1 (VCC), U1001.5 (VCC), U1002.4 (VCC), U1003.1 (VCC), U1003.5 (VCC)
- new net GND: C1001.2, C1002.2, C1003.2, R1001.2, R1003.2, SW1001.1, U1001.2 (GND), U1001.3 (GND), U1002.1 (GND), U1003.2 (GND), U1003.3 (GND)
- new net GPIO_LED_1: R1001.1, U1001.6
- new net GPIO_LED_2: R1003.1, U1003.6
- new net ~GPIO_SW: R1005.2, U1002.3 (OUT)

Commit message: Populated digi-key pn's
Parts:
- C1001, C1002, C1003: Digi-Key PN (none) -> 490-10701-1-ND
- D1001, D1002: footprint LEDs:LED_0603 -> LEDs:LED_0402; Digi-Key PN (none) -> 1497-1219-1-ND
- R1001, R1003, R1005: Digi-Key PN (none) -> RMCF0402FT10K0CT-ND
- R1002, R1004: Digi-Key PN (none) -> 541-1.00KLCT-ND
- U1002: Digi-Key PN (none) -> MAX6816EUS+TCT-ND
Changed lines of the file:
@@
 F 2 "Capacitors_SMD:C_0402" H 2808 1750 50  0001 C CNN
 F 3 "" H 2795 2000 50  0001 C CNN
-F 4 "" H 3195 2400 60  0001 C CNN "Digi-Key PN"
+F 4 "490-10701-1-ND" H 3195 2400 60  0001 C CNN "Digi-Key PN"
 F 5 "0402" H 2620 2000 50  0000 R CNN "display_footprint"
 F 6 "50V" H 2620 1900 50  0000 R CNN "Voltage"
@@
 F 0 "D1001" V 3489 2203 50  0000 R CNN
 F 1 "Green" V 3398 2203 50  0000 R CNN
-F 2 "LEDs:LED_0603" H 3450 2320 50  0001 C CNN
+F 2 "LEDs:LED_0402" H 3450 2320 50  0001 C CNN
 F 3 "~" H 3450 2320 50  0001 C CNN
-F 4 "" H -1710 -4000 50  0001 C CNN "Digi-Key PN"
+F 4 "1497-1219-1-ND" H -1710 -4000 50  0001 C CNN "Digi-Key PN"
 	1    3450 2320
 	0    -1   -1   0
@@
 F 5 "1%" H 3520 2020 50  0000 L CNN "Tolerance"
 F 6 "1/16W" H 3520 1950 50  0000 L CNN "Wattage"
-F 7 "" H 3750 2420 60  0001 C CNN "Digi-Key PN"
+F 7 "541-1.00KLCT-ND" H 3750 2420 60  0001 C CNN "Digi-Key PN"
 	1    3450 2020
 	-1   0    0    -1
@@
 F 5 "1%" H 2400 2820 50  0000 L CNN "Tolerance"
 F 6 "1/16W" H 2400 2750 50  0000 L CNN "Wattage"
-F 7 "" H 2330 2820 50  0001 C CNN "Digi-Key PN"
+F 7 "RMCF0402FT10K0CT-ND" H 2330 2820 50  0001 C CNN "Digi-Key PN"
 	1    2330 2820
 	-1   0    0    -1
@@
 F 2 "Capacitors_SMD:C_0402" H 4918 1750 50  0001 C CNN
 F 3 "" H 4905 2000 50  0001 C CNN
-F 4 "" H 5305 2400 60  0001 C CNN "Digi-Key PN"
+F 4 "490-10701-1-ND" H 5305 2400 60  0001 C CNN "Digi-Key PN"
 F 5 "0402" H 4730 2000 50  0000 R CNN "display_footprint"
 F 6 "50V" H 4730 1900 50  0000 R CNN "Voltage"
@@
 F 0 "D1002" V 5599 2203 50  0000 R CNN
 F 1 "Green" V 5508 2203 50  0000 R CNN
-F 2 "LEDs:LED_0603" H 5560 2320 50  0001 C CNN
+F 2 "LEDs:LED_0402" H 5560 2320 50  0001 C CNN
 F 3 "~" H 5560 2320 50  0001 C CNN
-F 4 "" H 400 -4000 50  0001 C CNN "Digi-Key PN"
+F 4 "1497-1219-1-ND" H 400 -4000 50  0001 C CNN "Digi-Key PN"
 	1    5560 2320
 	0    -1   -1   0
@@
 F 5 "1%" H 5630 2020 50  0000 L CNN "Tolerance"
 F 6 "1/16W" H 5630 1950 50  0000 L CNN "Wattage"
-F 7 "" H 5860 2420 60  0001 C CNN "Digi-Key PN"
+F 7 "541-1.00KLCT-ND" H 5860 2420 60  0001 C CNN "Digi-Key PN"
 	1    5560 2020
 	-1   0    0    -1
@@
 F 5 "1%" H 4510 2820 50  0000 L CNN "Tolerance"
 F 6 "1/16W" H 4510 2750 50  0000 L CNN "Wattage"
-F 7 "" H 4440 2820 50  0001 C CNN "Digi-Key PN"
+F 7 "RMCF0402FT10K0CT-ND" H 4440 2820 50  0001 C CNN "Digi-Key PN"
 	1    4440 2820
 	-1   0    0    -1
@@
 F 2 "Package_TO_SOT_SMD:SOT-143" H 5580 4870 50  0001 C CNN
 F 3 "https://datasheets.maximintegrated.com/en/ds/1896.pdf" H 4930 5320 50  0001 C CNN
+F 4 "MAX6816EUS+TCT-ND" H 4930 5320 50  0001 C CNN "Digi-Key PN"
 	1    4930 5320
 	1    0    0    -1
@@
 F 5 "1%" H 5760 5090 50  0000 L CNN "Tolerance"
 F 6 "1/16W" H 5760 5020 50  0000 L CNN "Wattage"
-F 7 "" H 5690 5090 50  0001 C CNN "Digi-Key PN"
+F 7 "RMCF0402FT10K0CT-ND" H 5690 5090 50  0001 C CNN "Digi-Key PN"
 	1    5690 5090
 	-1   0    0    -1
@@
 F 2 "Capacitors_SMD:C_0402" H 4518 4260 50  0001 C CNN
 F 3 "" H 4505 4510 50  0001 C CNN
-F 4 "" H 4905 4910 60  0001 C CNN "Digi-Key PN"
+F 4 "490-10701-1-ND" H 4905 4910 60  0001 C CNN "Digi-Key PN"
 F 5 "0402" H 4330 4510 50  0000 R CNN "display_footprint"
 F 6 "50V" H 4330 4410 50  0000 R CNN "Voltage"
