File: hdw/PIC32MZ_ETH_Demo/PIC32MZ_ETH_Demo.kicad_pcb (KiCad board)
At the start: 2 copper layers, 217 parts, among them J1201 USB_B_Mini, J201 +12V IN, J401 PICKIT3, J901 RJ45_Amphenol_RJMG1BD3B8K1ANR, Q401 BSS214NW, Q801 BSS214NW, SW1001 GPIO_SW, SW401 MRST, U1001 74LVC1G97, U1002 MAX6816, U1003 74LVC1G97, U1101 ISO7321C, U1201 TLV6700, U1202 FT234XD, U1203 TPD3S014DBVR, U1301 74LVC1G97, U1302 74LVC1G97, U1401 74LVC1G97, U1402 74LVC1G97, U1403 74LVC1G97, U1404 74LVC1G97, U1405 74LVC1G97, U1406 74LVC1G97, U301 TPS62130, U601 PIC32MZ2048EFG100_IPT, U801 TLV70012, U802 LAN8720A, X701 ASE-8.000MHz, X702 ECS-327KE, X801 ASE-25.000MHz

Commit message: Added BOM, finished arranging parts
Parts:
- C1001, C1002, C1003, C1301, C1401, C1402, C1403, C1404, C1405, C1406, C802, C803, C805, C809, L801, R1005, R801, R802, R804, R806, R807, R819, R820, R905, R906: moved to B.Cu
- moved U1404 189.7 mm to (256.7, 44.2)
- moved D1404 184.1 mm to (259.6, 45.2)
- moved R1409 183.3 mm to (259.6, 44.2)
- moved R1407 180.6 mm to (259.6, 43.2)
- moved C1404 178.3 mm to (256.7, 44.2), turned to 180 degrees
- moved U1406 172.0 mm to (248.7, 53.7)
- moved D1403 171.5 mm to (245.4, 45.4)
- moved U1403 170.4 mm to (242.4, 44.4)
- moved R1412 169.7 mm to (251.5, 53.7)
- moved C1406 168.4 mm to (248.7, 53.7), turned to 180 degrees
- moved R1404 166.7 mm to (245.4, 43.4)
- moved C1403 165.5 mm to (242.4, 44.4), turned to 180 degrees
- moved R1411 165.4 mm to (251.5, 52.7)
- moved D1406 165.0 mm to (251.5, 54.7)
- moved U1402 163.1 mm to (230.8, 44.4)
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Other:
- board text added: "+1.2VETH"
- board text added: "+3.3VAETH"

Commit message: Finished board layout
Parts:
- removed H1506, H1507, H1508: MountingHole, MountingHole:MountingHole_3mm
- added G***: PIC32_Logo, Custom Footprints Library:PIC32_Logo, F.Cu at (161.6, 75.9)
- added G***: Microchip_Logo, Custom Footprints Library:Microchip_Logo, B.Cu at (151.6, 65.8)
- added G***: Microchip_Logo, Custom Footprints Library:Microchip_Logo, F.Cu at (151.6, 65.8)
- added G***: Owl_1_Logo, Custom Footprints Library:Owl_1_Logo, B.Cu at (131.2, 63.5)
- added REF**: Symbol_Barrel_Polarity, Symbol:Symbol_Barrel_Polarity, F.Cu at (196.0, 46.1)
- moved C1102 160.0 mm to (120.9, 53.0)
- moved C1103 160.0 mm to (116.1, 54.9)
- moved C1203 160.0 mm to (110.4, 58.0)
- moved C1206 160.0 mm to (110.0, 50.7)
- moved C1210 160.0 mm to (105.1, 49.8)
- moved D1201 160.0 mm to (111.8, 51.4)
- moved J1201 160.0 mm to (100.1, 54.3)
- moved L1201 160.0 mm to (105.1, 51.8)
- moved L1202 160.0 mm to (105.1, 57.0)
- moved R1201 160.0 mm to (108.4, 49.7)
- moved R1202 160.0 mm to (106.2, 59.6)
- moved R1205 160.0 mm to (110.4, 56.1)
- moved R1208 160.0 mm to (111.8, 49.5)
- moved R1302 160.0 mm to (111.9, 54.4)
- moved U1101 160.0 mm to (120.9, 53.0)
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Connections:
- U601 pad 10: Net-(U601-Pad10) -> Reset_LED
- U601 pad 100: CPU_Exception_LED -> Net-(U601-Pad100)
- U601 pad 11: Net-(U601-Pad11) -> Heartbeat_LED
- U601 pad 17: GPIO_LED_1 -> Net-(U601-Pad17)
- U601 pad 3: Other_Error_LED -> Net-(U601-Pad3)
- U601 pad 38: GPIO_LED_2 -> Net-(U601-Pad38)
- U601 pad 43: ETH_PHY_CLKIN_EN -> Net-(U601-Pad43)
- U601 pad 44: ETH_PHY_RESET -> ~GPIO_SW
- U601 pad 57: Net-(U601-Pad57) -> GPIO_LED_2
- U601 pad 58: Net-(U601-Pad58) -> GPIO_LED_1
- U601 pad 59: ~GPIO_SW -> Net-(U601-Pad59)
- U601 pad 6: Net-(U601-Pad6) -> ETH_Error_LED
- U601 pad 60: Net-(U601-Pad60) -> ETH_PHY_RESET
- U601 pad 7: Net-(U601-Pad7) -> Other_Error_LED
- U601 pad 8: Net-(U601-Pad8) -> USB_Error_LED
- U601 pad 81: Net-(U601-Pad81) -> ETH_PHY_CLKIN_EN
- U601 pad 9: Net-(U601-Pad9) -> CPU_Exception_LED
- U601 pad 91: Heartbeat_LED -> Net-(U601-Pad91)
- U601 pad 94: Reset_LED -> Net-(U601-Pad94)
- U601 pad 98: USB_Error_LED -> Net-(U601-Pad98)
- U601 pad 99: ETH_Error_LED -> Net-(U601-Pad99)
Routing:
- net +3V3: track 0.00 -> 88.7 mm, vias 0 -> 45
- net GND: track 0.00 -> 88.3 mm, vias 0 -> 84
- net POS3P3_PGOOD: track 0.00 -> 77.7 mm, vias 0 -> 3
- net PHY_LED1: track 0.00 -> 51.1 mm, vias 0 -> 1
- net ETH_RMII_RXD0: track 0.00 -> 40.6 mm, vias 0 -> 2
- net ETH_RMII_RXD1: track 0.00 -> 40.5 mm, vias 0 -> 2
- net ETH_RMII_TXD1: track 0.00 -> 39.3 mm, vias 0 -> 2
- net USB_UART_TX: track 0.00 -> 38.1 mm, vias 0 -> 3
- net ~MCLR: track 0.00 -> 36.8 mm
- net ETH_RMII_REFCLK: track 0.00 -> 36.6 mm, vias 0 -> 2
- net ETH_RMII_TXD0: track 0.00 -> 36.2 mm, vias 0 -> 2
- net PHY_LED2: track 0.00 -> 35.1 mm, vias 0 -> 1
- net ETH_RMII_RXERR: track 0.00 -> 34.1 mm, vias 0 -> 2
- net ETH_RMII_CRSDV: track 0.00 -> 32.9 mm, vias 0 -> 2
- net ETH_PHY_CLKIN_EN: track 0.00 -> 32.8 mm
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- added copper zone on F.Cu, net +12V
- added copper zone on B.Cu, net +3.3VA_ETH
- added copper zone on F.Cu, net +3V3
- added copper zone on PWR, net +3V3
- added copper zone on PWR, net +5V_USB
- added copper zone on GND, net GND
- added copper zone on GND, net GND_USB
- added copper zone on F.Cu, net Net-(L301-Pad1)
Other:
- board outline added: 108.9 x 39.5 mm
- copper layers 2 -> 4
- net class Default: clearance 0.2 -> 0.1524; trace_width 0.25 -> 0.254; via_dia 0.8 -> 0.508; via_drill 0.4 -> 0.254
- net class Power added: clearance 0.1524, trace_width 0.635, via_dia 0.508, via_drill 0.254
- net class Signal added: clearance 0.1524, trace_width 0.254, via_dia 0.508, via_drill 0.254
- rule trace_clearance: 0.2 -> 0.1524
- rule trace_min: 0.2 -> 0.0508
- rule via_min_drill: 0.3 -> 0.199898
- board text added: "+"
- board text added: "+12VIN NO PROTECTION"
- board text added: "+3.3V PGOOD"
- board text added: "-"
- board text added: "CPU Trap"
- board text added: "ETH Error"
- board text added: "Heart Beat"
- board text added: "MRST"
- board text added: "Other Error"
- board text added: "PIC KIT 3"
- board text added: "PIC32MZ ETH DEMO"
- board text added: "Reset/ Prog"
- board text added: "USB Error"
